File: pcb/usb-and-battery.kicad_sch (KiCad schematic)
At the start: 29 parts, among them J4 USB_C_Receptacle_USB2.0, J7 Conn_01x02, Q1 DMG3401LSN, Q2 DMG3418L, Q3 DMG3418L, SW1 SW_SPST, U147 AP2112K-3.3, U149 74LVC1G17GW,125, U151 74LVC1G80, U152 BQ297xy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

Commit message: Remove battery power option
- This device needs user IO
- Battery power means there would need to be a touch screen or wireless
  connection. Too complex.
Parts:
- removed C2: 10uF, Capacitor_SMD:C_0805_2012Metric, symbol Device:C
- removed C2: 0.1uF, Capacitor_SMD:C_0402_1005Metric, symbol Device:C
- removed D4: MBR540, symbol Device:D_Schottky
- removed J7: Conn_01x02, Connector_JST:JST_PH_S2B-PH-SM4-TB_1x02-1MP_P2.00mm_Horizontal, symbol Connector_Generic:Conn_01x02
- removed Q1: DMG3401LSN, Package_TO_SOT_SMD:SOT-23, symbol Transistor_FET:DMG2301L
- removed Q2, Q3: DMG3418L, Package_TO_SOT_SMD:SOT-23, symbol Transistor_FET:DMG3414U
- removed R2: 2.2k, symbol Device:R_US
- removed R2 (x2): 10k, symbol Device:R_US
- removed R2: 330, symbol Device:R_US
- removed R2: 4.7k, symbol Device:R_US
- removed SW1: SW_SPST, symbol Switch:SW_SPST
- removed U152: BQ297xy, Package_SON:WSON-6_1.5x1.5mm_P0.5mm, symbol Battery_Management:BQ297xy
- removed U153: MCP73831-2-OT, Package_TO_SOT_SMD:SOT-23-5, symbol Battery_Management:MCP73831-2-OT
- added R272: 10k, Resistor_SMD:R_0402_1005Metric, symbol Device:R_US
- added SW2: PBH2UEESNPNAGX, open-ephys:ESWITCH_PBH2UxxNAGX, symbol Switch:SW_DPDT_x2
- J4: value USB_C_Receptacle_USB2.0 -> USB4105; footprint (none) -> Connector_USB:USB_C_Receptacle_GCT_USB4105-xx-A_16P_TopMnt_Horizontal
- R148, R149, R265, R269: renamed from R2; footprint (none) -> Resistor_SMD:R_0402_1005Metric
- renumbered C2 to C273, C2 to C274, C2 to C275, C2 to C276, C2 to C277, C2 to C278
Connections:
- net VPP is gone; now on net VBUS: C273.1, C275.1, C276.1, U147.1 (VIN), U149.5 (VCC), U151.5 (VCC)
- net GND: now also SW2.1 (A), SW2.4 (A)
- net VBUS: now also R272.1
- net at U149.2: now also SW2.2 (B), SW2.5 (B)
- new net: R272.2, SW2.3 (C), SW2.6 (C)
Other:
- note added: "Compatible caps * 1R (round; 9mm len. 5 mm diam) * 1C (rectangle) * 1S (square) Throw: * 2 mm to lock * 3 mm max"
- moved on the sheet: C273, C274, C275, C276, C277, C278, J4, R148, R149, R265, R269, U147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
