File: pcb/signal-routing.kicad_sch (KiCad schematic)
At the start: 42 parts, among them U10 SN74LVC1G3157DCKR, U12 SN74LVC1G3157DCKR, U13 SN74LVC1G3157DCKR, U14 SN74LVC1G3157DCKR, U15 SN74LVC1G3157DCKR, U2 SN74LVC1G3157DCKR, U3 SN74LVC1G3157DCKR, U4 SN74HCS595, U8 SN74LVC1G3157DCKR

Commit message: Remove battery power option
- This device needs user IO
- Battery power means there would need to be a touch screen or wireless
  connection. Too complex.
Parts:
- R1: value 1M -> 100k
- R124, R169, R2, R201, R233, R42, R84: renamed from R1; value 1M -> 100k
- renumbered R3 to R125, R3 to R170, R3 to R202, R3 to R234, R3 to R43, R3 to R5, R3 to R85

Commit message: Finished schematic, started routing
- There is a 8-channel motif that will need to be copied 16x on the
  board. I'm not sure the most efficient way to do this.
Parts:
- renumbered C1 to C63, C25 to C65, C2 to C66, C128 to C67, C4 to C68, C26 to C69, C6 to C70, C30 to C71, C162 to C72, C14 to C73, C27 to C74, C64 to C75, C191 to C76, C18 to C77, C28 to C78, C94 to C79, C225 to C80, R1 to R55, R124 to R56, R3 to R57, R125 to R58, R2 to R59, R169 to R60, R5 to R61, R170 to R62, R42 to R63, R201 to R64, R43 to R65, R202 to R66, R84 to R67, R233 to R68, R85 to R69, R234 to R70, U2 to U38, U12 to U39, U3 to U40, U13 to U41, U4 to U42, U8 to U43, U14 to U44, U10 to U45, U15 to U46

Commit message: Motif is repeated
- some components are grouped by function
- components are roughly organized within groups
Parts:
- renumbered C70 to C100, C66 to C84, C71 to C85, C75 to C86, C79 to C87, C63 to C88, C68 to C89, C73 to C90, C77 to C91, C67 to C92, C72 to C93, C76 to C94, C80 to C95, C65 to C96, C69 to C97, C74 to C98, C78 to C99, R57 to R70, R61 to R71, R65 to R72, R69 to R73, R55 to R74, R59 to R75, R63 to R76, R67 to R77, R58 to R78, R62 to R79, R66 to R80, R70 to R81, R56 to R82, R60 to R83, R64 to R84, R68 to R85, U38 to U39, U43 to U41, U45 to U42, U39 to U43, U41 to U44, U44 to U45, U42 to U47
Connections:
- net E_{4}: now also R78.1, R82.2; no longer R81.1, R85.2
- net E_{5}: now also R79.1, R83.2; no longer R80.1, R84.2
- net E_{6}: now also R80.1, R84.2; no longer R79.1, R83.2
- net E_{7}: now also R81.1, R85.2; no longer R78.1, R82.2
- net S_{4}: now also U43.6; no longer U46.6
- net S_{5}: now also U44.6; no longer U45.6
- net S_{6}: now also U45.6; no longer U44.6
- net S_{7}: now also U46.6; no longer U43.6
