File: pcb/signal-routing.kicad_sch (KiCad schematic)
At the start: 26 parts, among them U3 FSA553, U4 FSA553, U5 FSA553, U6 FSA553, U7 SN74HC595PWR

Commit message: Revision G candidate
- Fix flipped power/ground connections on U84
- VCC is now 3.0V
- Address issues with parasitic voltage feedthrough on FSA533
- Completely redesign test signal analog section with much
  improved noise, THD, etc and implicit low THD input protection on the
  external input.
Parts:
- R15, R16, R17, R18, R23, R24, R25, R26: value 100k -> 19.8k; LCSC C852472 -> (none)
Changed lines of the file:
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@@
 		(title "Extracellular Electrophysiology Test Board")
 		(date "2025-03-20")
-		(rev "F")
+		(rev "G")
 		(company "Open Ephys, Inc")
 		(comment 1 "Jonathan P. Newman")
@@
 			)
 		)
-		(property "Value" "100k"
+		(property "Value" "19.8k"
 			(at 135.89 165.1 90)
 			(effects
@@
 			)
 		)
-		(property "LCSC" "C852472"
+		(property "LCSC" ""
 			(at 135.89 167.64 90)
 			(effects
@@
 			)
 		)
-		(property "Value" "100k"
+		(property "Value" "19.8k"
 			(at 62.23 81.28 90)
 			(effects
@@
 			)
 		)
-		(property "LCSC" "C852472"
+		(property "LCSC" ""
 			(at 62.23 83.82 90)
 			(effects
@@
 			)
 		)
-		(property "Value" "100k"
+		(property "Value" "19.8k"
 			(at 62.23 39.37 90)
 			(effects
@@
 			)
 		)
-		(property "LCSC" "C852472"
+		(property "LCSC" ""
 			(at 62.23 41.91 90)
 			(effects
@@
 			)
 		)
-		(property "Value" "100k"
+		(property "Value" "19.8k"
 			(at 135.89 125.73 90)
 			(effects
@@
 			)
 		)
-		(property "LCSC" "C852472"
+		(property "LCSC" ""
 			(at 135.89 128.27 90)
 			(effects
@@
 			)
 		)
-		(property "Value" "100k"
+		(property "Value" "19.8k"
 			(at 62.23 165.1 90)
 			(effects
@@
 			)
 		)
-		(property "LCSC" "C852472"
+		(property "LCSC" ""
 			(at 62.23 167.64 90)
 			(effects
@@
 			)
 		)
-		(property "Value" "100k"
+		(property "Value" "19.8k"
 			(at 62.23 125.73 90)
 			(effects
@@
 			)
 		)
-		(property "LCSC" "C852472"
+		(property "LCSC" ""
 			(at 62.23 128.27 90)
 			(effects
@@
 			)
 		)
-		(property "Value" "100k"
+		(property "Value" "19.8k"
 			(at 135.89 39.37 90)
 			(effects
@@
 			)
 		)
-		(property "LCSC" "C852472"
+		(property "LCSC" ""
 			(at 135.89 41.91 90)
 			(effects
@@
 			)
 		)
-		(property "Value" "100k"
+		(property "Value" "19.8k"
 			(at 135.89 81.28 90)
 			(effects
@@
 			)
 		)
-		(property "LCSC" "C852472"
+		(property "LCSC" ""
 			(at 135.89 83.82 90)
 			(effects

Commit message: Update PCB component part numbers
Replace and fill missing MPN and OEPSPN properties.
Parts:
- R15, R16, R17, R18, R23, R24, R25, R26: MPN RG1005P-104-B-T5 -> RN73R1ETTP1982B25; OEPSPN OEPS020175 -> OEPS020208
- U3, U4, U5, U6: MPN (none) -> FSA553UCX; OEPSPN (none) -> OEPS080198
- U7: MPN SN74HCS595PWR -> SN74HC595PWR; OEPSPN OEPS080159 -> OEPS080200
Changed lines of the file:
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@@
 			)
 		)
+		(property "MPN" "FSA553UCX"
+			(at 152.4 165.1 0)
+			(effects
+				(font
+					(size 1.27 1.27)
+				)
+				(hide yes)
+			)
+		)
+		(property "OEPSPN" "OEPS080198"
+			(at 152.4 165.1 0)
+			(effects
+				(font
+					(size 1.27 1.27)
+				)
+				(hide yes)
+			)
+		)
 		(pin "C1"
 		)
@@
 			)
 		)
+		(property "MPN" "FSA553UCX"
+			(at 77.47 81.28 0)
+			(effects
+				(font
+					(size 1.27 1.27)
+				)
+				(hide yes)
+			)
+		)
+		(property "OEPSPN" "OEPS080198"
+			(at 77.47 81.28 0)
+			(effects
+				(font
+					(size 1.27 1.27)
+				)
+				(hide yes)
+			)
+		)
 		(pin "C1"
 		)
@@
 			)
 		)
-		(property "MPN" "RG1005P-104-B-T5"
+		(property "MPN" "RN73R1ETTP1982B25"
 			(at 135.89 167.64 0)
 			(effects
@@
 			)
 		)
-		(property "OEPSPN" "OEPS020175"
+		(property "OEPSPN" "OEPS020208"
 			(at 135.89 167.64 0)
 			(effects
@@
 			)
 		)
-		(property "MPN" "RG1005P-104-B-T5"
+		(property "MPN" "RN73R1ETTP1982B25"
 			(at 62.23 83.82 0)
 			(effects
@@
 			)
 		)
-		(property "OEPSPN" "OEPS020175"
+		(property "OEPSPN" "OEPS020208"
 			(at 62.23 83.82 0)
 			(effects
@@
 			)
 		)
-		(property "MPN" "RG1005P-104-B-T5"
+		(property "MPN" "RN73R1ETTP1982B25"
 			(at 62.23 41.91 0)
 			(effects
@@
 			)
 		)
-		(property "OEPSPN" "OEPS020175"
+		(property "OEPSPN" "OEPS020208"
 			(at 62.23 41.91 0)
 			(effects
@@
 			)
 		)
+		(property "MPN" "FSA553UCX"
+			(at 77.47 125.73 0)
+			(effects
+				(font
+					(size 1.27 1.27)
+				)
+				(hide yes)
+			)
+		)
+		(property "OEPSPN" "OEPS080198"
+			(at 77.47 125.73 0)
+			(effects
+				(font
+					(size 1.27 1.27)
+				)
+				(hide yes)
+			)
+		)
 		(pin "C1"
 		)
@@
 			)
 		)
-		(property "MPN" "SN74HCS595PWR"
+		(property "MPN" "SN74HC595PWR"
 			(at 215.9 90.17 0)
 			(effects
@@
 			)
 		)
-		(property "OEPSPN" "OEPS080159"
+		(property "OEPSPN" "OEPS080200"
 			(at 215.9 90.17 0)
 			(effects
@@
 			)
 		)
-		(property "MPN" "RG1005P-104-B-T5"
+		(property "MPN" "RN73R1ETTP1982B25"
 			(at 135.89 128.27 0)
 			(effects
@@
 			)
 		)
-		(property "OEPSPN" "OEPS020175"
+		(property "OEPSPN" "OEPS020208"
 			(at 135.89 128.27 0)
 			(effects
@@
 			)
 		)
-		(property "MPN" "RG1005P-104-B-T5"
+		(property "MPN" "RN73R1ETTP1982B25"
 			(at 62.23 167.64 0)
 			(effects
@@
 			)
 		)
-		(property "OEPSPN" "OEPS020175"
+		(property "OEPSPN" "OEPS020208"
 			(at 62.23 167.64 0)
 			(effects
@@
 			)
 		)
-		(property "MPN" "RG1005P-104-B-T5"
+		(property "MPN" "RN73R1ETTP1982B25"
 			(at 62.23 128.27 0)
 			(effects
@@
 			)
 		)
-		(property "OEPSPN" "OEPS020175"
+		(property "OEPSPN" "OEPS020208"
 			(at 62.23 128.27 0)
 			(effects
@@
 			)
 		)
+		(property "MPN" "FSA553UCX"
+			(at 152.4 125.73 0)
+			(effects
+				(font
+					(size 1.27 1.27)
+				)
+				(hide yes)
+			)
+		)
+		(property "OEPSPN" "OEPS080198"
+			(at 152.4 125.73 0)
+			(effects
+				(font
+					(size 1.27 1.27)
+				)
+				(hide yes)
+			)
+		)
 		(pin "C1"
 		)
@@
 			)
 		)
-		(property "MPN" "RG1005P-104-B-T5"
+		(property "MPN" "RN73R1ETTP1982B25"
 			(at 135.89 41.91 0)
 			(effects
@@
 			)
 		)
-		(property "OEPSPN" "OEPS020175"
+		(property "OEPSPN" "OEPS020208"
 			(at 135.89 41.91 0)
 			(effects
@@
 			)
 		)
+		(property "MPN" "FSA553UCX"
+			(at 77.47 165.1 0)
+			(effects
+				(font
+					(size 1.27 1.27)
+				)
+				(hide yes)
+			)
+		)
+		(property "OEPSPN" "OEPS080198"
+			(at 77.47 165.1 0)
+			(effects
+				(font
+					(size 1.27 1.27)
+				)
+				(hide yes)
+			)
+		)
 		(pin "C1"
 		)
@@
 			)
 		)
+		(property "MPN" "FSA553UCX"
+			(at 152.4 39.37 0)
+			(effects
+				(font
+					(size 1.27 1.27)
+				)
+				(hide yes)
+			)
+		)
+		(property "OEPSPN" "OEPS080198"
+			(at 152.4 39.37 0)
+			(effects
+				(font
+					(size 1.27 1.27)
+				)
+				(hide yes)
+			)
+		)
 		(pin "C1"
 		)
@@
 			)
 		)
+		(property "MPN" "FSA553UCX"
+			(at 77.47 39.37 0)
+			(effects
+				(font
+					(size 1.27 1.27)
+				)
+				(hide yes)
+			)
+		)
+		(property "OEPSPN" "OEPS080198"
+			(at 77.47 39.37 0)
+			(effects
+				(font
+					(size 1.27 1.27)
+				)
+				(hide yes)
+			)
+		)
 		(pin "C1"
 		)
@@
 			)
 		)
-		(property "MPN" "RG1005P-104-B-T5"
+		(property "MPN" "RN73R1ETTP1982B25"
 			(at 135.89 83.82 0)
 			(effects
@@
 			)
 		)
-		(property "OEPSPN" "OEPS020175"
+		(property "OEPSPN" "OEPS020208"
 			(at 135.89 83.82 0)
 			(effects
@@
 			(effects
 				(font
+					(size 1.27 1.27)
+				)
+				(hide yes)
+			)
+		)
+		(property "MPN" "FSA553UCX"
+			(at 152.4 81.28 0)
+			(effects
+				(font
+					(size 1.27 1.27)
+				)
+				(hide yes)
+			)
+		)
+		(property "OEPSPN" "OEPS080198"
+			(at 152.4 81.28 0)
+			(effects
+				(font

Commit message: Updated OEPS PN and regenerated BOM and PnP files
Parts:
- U3, U4, U5, U6: value FSA553 -> FSA553UCX; LCSC (none) -> C605183
Changed lines of the file:
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@@
 			)
 		)
-		(property "Value" "FSA553"
+		(property "Value" "FSA553UCX"
 			(at 152.4 157.48 0)
 			(effects
@@
 			)
 		)
+		(property "LCSC" "C605183 "
+			(at 152.4 165.1 0)
+			(effects
+				(font
+					(size 1.27 1.27)
+				)
+				(hide yes)
+			)
+		)
 		(pin "C1"
 		)
@@
 			)
 		)
-		(property "Value" "FSA553"
+		(property "Value" "FSA553UCX"
 			(at 77.47 73.66 0)
 			(effects
@@
 			)
 		)
+		(property "LCSC" "C605183 "
+			(at 77.47 81.28 0)
+			(effects
+				(font
+					(size 1.27 1.27)
+				)
+				(hide yes)
+			)
+		)
 		(pin "C1"
 		)
@@
 			)
 		)
-		(property "Value" "FSA553"
+		(property "Value" "FSA553UCX"
 			(at 70.612 115.316 0)
 			(effects
@@
 			)
 		)
+		(property "LCSC" "C605183 "
+			(at 77.47 125.73 0)
+			(effects
+				(font
+					(size 1.27 1.27)
+				)
+				(hide yes)
+			)
+		)
 		(pin "C1"
 		)
@@
 			)
 		)
-		(property "Value" "FSA553"
+		(property "Value" "FSA553UCX"
 			(at 146.05 115.824 0)
 			(effects
@@
 			)
 		)
+		(property "LCSC" "C605183 "
+			(at 152.4 125.73 0)
+			(effects
+				(font
+					(size 1.27 1.27)
+				)
+				(hide yes)
+			)
+		)
 		(pin "C1"
 		)
@@
 			)
 		)
-		(property "Value" "FSA553"
+		(property "Value" "FSA553UCX"
 			(at 77.47 157.48 0)
 			(effects
@@
 			)
 		)
+		(property "LCSC" "C605183 "
+			(at 77.47 165.1 0)
+			(effects
+				(font
+					(size 1.27 1.27)
+				)
+				(hide yes)
+			)
+		)
 		(pin "C1"
 		)
@@
 			)
 		)
-		(property "Value" "FSA553"
+		(property "Value" "FSA553UCX"
 			(at 146.304 29.464 0)
 			(effects
@@
 			)
 		)
+		(property "LCSC" "C605183 "
+			(at 152.4 39.37 0)
+			(effects
+				(font
+					(size 1.27 1.27)
+				)
+				(hide yes)
+			)
+		)
 		(pin "C1"
 		)
@@
 			)
 		)
-		(property "Value" "FSA553"
+		(property "Value" "FSA553UCX"
 			(at 70.612 28.956 0)
 			(effects
@@
 			)
 		)
+		(property "LCSC" "C605183 "
+			(at 77.47 39.37 0)
+			(effects
+				(font
+					(size 1.27 1.27)
+				)
+				(hide yes)
+			)
+		)
 		(pin "C1"
 		)
@@
 			)
 		)
-		(property "Value" "FSA553"
+		(property "Value" "FSA553UCX"
 			(at 152.4 73.66 0)
 			(effects
@@
 			(at 152.4 81.28 0)
 			(effects
+				(font
+					(size 1.27 1.27)
+				)
+				(hide yes)
+			)
+		)
+		(property "LCSC" "C605183 "
+			(at 152.4 81.28 0)
+			(effects
