File: pcb/signal-routing.kicad_sch (KiCad schematic)
At the start: 26 parts, among them U3 FSA553UCX, U4 FSA553UCX, U5 FSA553UCX, U6 FSA553UCX, U7 SN74HC595PWR

Commit message: Rev. G production candidate
- Finished LCSC part numbers
- Generated final gerbers
Parts:
- R15, R16, R17, R18, R23, R24, R25, R26: LCSC (none) -> C2535118
Changed lines of the file:
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@@
 			)
 		)
-		(property "LCSC" ""
+		(property "LCSC" "C2535118"
 			(at 135.89 167.64 90)
 			(effects
@@
 			)
 		)
-		(property "LCSC" ""
+		(property "LCSC" "C2535118"
 			(at 62.23 83.82 90)
 			(effects
@@
 			)
 		)
-		(property "LCSC" ""
+		(property "LCSC" "C2535118"
 			(at 62.23 41.91 90)
 			(effects
@@
 			)
 		)
-		(property "LCSC" ""
+		(property "LCSC" "C2535118"
 			(at 135.89 128.27 90)
 			(effects
@@
 			)
 		)
-		(property "LCSC" ""
+		(property "LCSC" "C2535118"
 			(at 62.23 167.64 90)
 			(effects
@@
 			)
 		)
-		(property "LCSC" ""
+		(property "LCSC" "C2535118"
 			(at 62.23 128.27 90)
 			(effects
@@
 			)
 		)
-		(property "LCSC" ""
+		(property "LCSC" "C2535118"
 			(at 135.89 41.91 90)
 			(effects
@@
 			)
 		)
-		(property "LCSC" ""
+		(property "LCSC" "C2535118"
 			(at 135.89 83.82 90)
 			(effects
