File: pcb/signal-routing.kicad_sch (KiCad schematic)
At the start: 26 parts, among them U3 FSA553UCX, U4 FSA553UCX, U5 FSA553UCX, U6 FSA553UCX, U7 SN74HC595PWR

Commit message: update revision to H
- Minor schematic fixes
- Update attenuator resistors to match rev. g values
- Update silkscreen to indicate revision H
Parts:
- R11, R12, R13, R14, R19, R20, R21, R22: value 200R -> 301R; LCSC C852625 -> C705632; MPN ERA-2AEB201X -> RT0402BRD07301RL
- R15, R16, R17, R18, R23, R24, R25, R26: value 19.8k -> 29.8k; LCSC C2535118 -> C2506693; MPN RN73R1ETTP1982B25 -> RN73R1ETTP2982B25; OEPSPN OEPS020208 -> OEPS020222

Commit message: Update part numbers
Replace OEPSPN 'OEPS020171' with 'OEPS020223'.
Correct component Value and MPN by adding a leading zero ('731000105' -> '0731000105').
Parts:
- R11, R12, R13, R14, R19, R20, R21, R22: OEPSPN OEPS020171 -> OEPS020223
Changed lines of the file:
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@@
 			)
 		)
-		(property "OEPSPN" "OEPS020171"
+		(property "OEPSPN" "OEPS020223"
 			(at 55.88 173.99 0)
 			(hide yes)
@@
 			)
 		)
-		(property "OEPSPN" "OEPS020171"
+		(property "OEPSPN" "OEPS020223"
 			(at 55.88 48.26 0)
 			(hide yes)
@@
 			)
 		)
-		(property "OEPSPN" "OEPS020171"
+		(property "OEPSPN" "OEPS020223"
 			(at 129.54 173.99 0)
 			(hide yes)
@@
 			)
 		)
-		(property "OEPSPN" "OEPS020171"
+		(property "OEPSPN" "OEPS020223"
 			(at 129.54 134.62 0)
 			(hide yes)
@@
 			)
 		)
-		(property "OEPSPN" "OEPS020171"
+		(property "OEPSPN" "OEPS020223"
 			(at 129.54 48.26 0)
 			(hide yes)
@@
 			)
 		)
-		(property "OEPSPN" "OEPS020171"
+		(property "OEPSPN" "OEPS020223"
 			(at 55.88 90.17 0)
 			(hide yes)
@@
 			)
 		)
-		(property "OEPSPN" "OEPS020171"
+		(property "OEPSPN" "OEPS020223"
 			(at 55.88 134.62 0)
 			(hide yes)
@@
 			)
 		)
-		(property "OEPSPN" "OEPS020171"
+		(property "OEPSPN" "OEPS020223"
 			(at 129.54 90.17 0)
 			(hide yes)

Commit message: Added 'Description' to all the components
Updated PCB accordingly.
Configured files for manufacturing generation according to standards.
Parts:
- C16, C17, C18, C19: OEPS Description (none) -> CAPACITOR: SMD CER 0402 10nF 25V ±10% X7R (OEPS H1 002) [GR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
- C20: OEPS Description (none) -> CAPACITOR: SMD CER 0402 100nF 25V ±10% X7R (OEPS H02 001) [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
- R11, R12, R13, R14, R19, R20, R21, R22: OEPS Description (none) -> RESISTOR: SMD 0402 301Ω ±0.1% 0.063W [RT0402BRD07301RL] [SM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
- R15, R16, R17, R18, R23, R24, R25, R26: OEPS Description (none) -> RESISTOR: SMD 0402 29.8kΩ ±0.1% 0.063W [RN73R1ETTP2982B25] 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
- U3, U4, U5, U6: OEPS Description (none) -> IC: AUDIO SWITCH SPST DUAL [FSA553UCX] [9-WLCSP]
- U7: OEPS Description (none) -> IC: 8-BIT SHIFT REGISTER [SN74HC595PWR] [16-TSSOP]
Changed lines of the file:
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@@
 			)
 		)
+		(property "OEPS Description" "IC:   AUDIO SWITCH SPST DUAL   [FSA553UCX] [9-WLCSP]" (at 152.4 165.1 0) (effects (font (size 1.27 1.27)) (hide yes)))
 	)
 	(symbol
@@
 			)
 		)
+		(property "OEPS Description" "IC:   AUDIO SWITCH SPST DUAL   [FSA553UCX] [9-WLCSP]" (at 77.47 81.28 0) (effects (font (size 1.27 1.27)) (hide yes)))
 	)
 	(symbol
@@
 			)
 		)
+		(property "OEPS Description" "RESISTOR:   SMD 0402 29.8kΩ ±0.1% 0.063W   [RN73R1ETTP2982B25] [SMD]" (at 135.89 167.64 0) (effects (font (size 1.27 1.27)) (hide yes)))
 	)
 	(symbol
@@
 			)
 		)
+		(property "OEPS Description" "CAPACITOR:   SMD CER 0402 10nF 25V ±10% X7R (OEPS H1 002)   [GRM155R71E103KA01D] [SMD]" (at 83.82 22.86 0) (effects (font (size 1.27 1.27)) (hide yes)))
 	)
 	(symbol
@@
 			)
 		)
+		(property "OEPS Description" "RESISTOR:   SMD 0402 301Ω ±0.1% 0.063W   [RT0402BRD07301RL] [SMD]" (at 55.88 173.99 0) (effects (font (size 1.27 1.27)) (hide yes)))
 	)
 	(symbol
@@
 			)
 		)
+		(property "OEPS Description" "RESISTOR:   SMD 0402 29.8kΩ ±0.1% 0.063W   [RN73R1ETTP2982B25] [SMD]" (at 62.23 83.82 0) (effects (font (size 1.27 1.27)) (hide yes)))
 	)
 	(symbol
@@
 			)
 		)
+		(property "OEPS Description" "RESISTOR:   SMD 0402 29.8kΩ ±0.1% 0.063W   [RN73R1ETTP2982B25] [SMD]" (at 62.23 41.91 0) (effects (font (size 1.27 1.27)) (hide yes)))
 	)
 	(symbol
@@
 			)
 		)
+		(property "OEPS Description" "RESISTOR:   SMD 0402 301Ω ±0.1% 0.063W   [RT0402BRD07301RL] [SMD]" (at 55.88 48.26 0) (effects (font (size 1.27 1.27)) (hide yes)))
 	)
 	(symbol
@@
 			)
 		)
+		(property "OEPS Description" "CAPACITOR:   SMD CER 0402 100nF 25V ±10% X7R (OEPS H02 001)   [C1005X7R1E104K050BB] [SMD]" (at 245.11 76.2 0) (effects (font (size 1.27 1.27)) (hide yes)))
 	)
 	(symbol
@@
 			)
 		)
+		(property "OEPS Description" "RESISTOR:   SMD 0402 301Ω ±0.1% 0.063W   [RT0402BRD07301RL] [SMD]" (at 129.54 173.99 0) (effects (font (size 1.27 1.27)) (hide yes)))
 	)
 	(symbol
@@
 			)
 		)
+		(property "OEPS Description" "CAPACITOR:   SMD CER 0402 10nF 25V ±10% X7R (OEPS H1 002)   [GRM155R71E103KA01D] [SMD]" (at 83.82 109.22 0) (effects (font (size 1.27 1.27)) (hide yes)))
 	)
 	(symbol
@@
 			)
 		)
+		(property "OEPS Description" "RESISTOR:   SMD 0402 301Ω ±0.1% 0.063W   [RT0402BRD07301RL] [SMD]" (at 129.54 134.62 0) (effects (font (size 1.27 1.27)) (hide yes)))
 	)
 	(symbol
@@
 			)
 		)
+		(property "OEPS Description" "IC:   AUDIO SWITCH SPST DUAL   [FSA553UCX] [9-WLCSP]" (at 77.47 125.73 0) (effects (font (size 1.27 1.27)) (hide yes)))
 	)
 	(symbol
@@
 			)
 		)
+		(property "OEPS Description" "CAPACITOR:   SMD CER 0402 10nF 25V ±10% X7R (OEPS H1 002)   [GRM155R71E103KA01D] [SMD]" (at 158.75 22.86 0) (effects (font (size 1.27 1.27)) (hide yes)))
 	)
 	(symbol
@@
 			)
 		)
+		(property "OEPS Description" "IC:   8-BIT SHIFT REGISTER   [SN74HC595PWR] [16-TSSOP]" (at 215.9 90.17 0) (effects (font (size 1.27 1.27)) (hide yes)))
 	)
 	(symbol
@@
 			)
 		)
+		(property "OEPS Description" "CAPACITOR:   SMD CER 0402 10nF 25V ±10% X7R (OEPS H1 002)   [GRM155R71E103KA01D] [SMD]" (at 158.75 109.22 0) (effects (font (size 1.27 1.27)) (hide yes)))
 	)
 	(symbol
@@
 			)
 		)
+		(property "OEPS Description" "RESISTOR:   SMD 0402 29.8kΩ ±0.1% 0.063W   [RN73R1ETTP2982B25] [SMD]" (at 135.89 128.27 0) (effects (font (size 1.27 1.27)) (hide yes)))
 	)
 	(symbol
@@
 			)
 		)
+		(property "OEPS Description" "RESISTOR:   SMD 0402 29.8kΩ ±0.1% 0.063W   [RN73R1ETTP2982B25] [SMD]" (at 62.23 167.64 0) (effects (font (size 1.27 1.27)) (hide yes)))
 	)
 	(symbol
@@
 			)
 		)
+		(property "OEPS Description" "RESISTOR:   SMD 0402 29.8kΩ ±0.1% 0.063W   [RN73R1ETTP2982B25] [SMD]" (at 62.23 128.27 0) (effects (font (size 1.27 1.27)) (hide yes)))
 	)
 	(symbol
@@
 			)
 		)
+		(property "OEPS Description" "RESISTOR:   SMD 0402 301Ω ±0.1% 0.063W   [RT0402BRD07301RL] [SMD]" (at 129.54 48.26 0) (effects (font (size 1.27 1.27)) (hide yes)))
 	)
 	(symbol
@@
 			)
 		)
+		(property "OEPS Description" "RESISTOR:   SMD 0402 301Ω ±0.1% 0.063W   [RT0402BRD07301RL] [SMD]" (at 55.88 90.17 0) (effects (font (size 1.27 1.27)) (hide yes)))
 	)
 	(symbol
@@
 			)
 		)
+		(property "OEPS Description" "IC:   AUDIO SWITCH SPST DUAL   [FSA553UCX] [9-WLCSP]" (at 152.4 125.73 0) (effects (font (size 1.27 1.27)) (hide yes)))
 	)
 	(symbol
@@
 			)
 		)
+		(property "OEPS Description" "RESISTOR:   SMD 0402 29.8kΩ ±0.1% 0.063W   [RN73R1ETTP2982B25] [SMD]" (at 135.89 41.91 0) (effects (font (size 1.27 1.27)) (hide yes)))
 	)
 	(symbol
@@
 			)
 		)
+		(property "OEPS Description" "IC:   AUDIO SWITCH SPST DUAL   [FSA553UCX] [9-WLCSP]" (at 77.47 165.1 0) (effects (font (size 1.27 1.27)) (hide yes)))
 	)
 	(symbol
@@
 			)
 		)
+		(property "OEPS Description" "IC:   AUDIO SWITCH SPST DUAL   [FSA553UCX] [9-WLCSP]" (at 152.4 39.37 0) (effects (font (size 1.27 1.27)) (hide yes)))
 	)
 	(symbol
@@
 			)
 		)
+		(property "OEPS Description" "IC:   AUDIO SWITCH SPST DUAL   [FSA553UCX] [9-WLCSP]" (at 77.47 39.37 0) (effects (font (size 1.27 1.27)) (hide yes)))
 	)
 	(symbol
@@
 			)
 		)
+		(property "OEPS Description" "RESISTOR:   SMD 0402 301Ω ±0.1% 0.063W   [RT0402BRD07301RL] [SMD]" (at 55.88 134.62 0) (effects (font (size 1.27 1.27)) (hide yes)))
 	)
 	(symbol
@@
 			)
 		)
+		(property "OEPS Description" "RESISTOR:   SMD 0402 29.8kΩ ±0.1% 0.063W   [RN73R1ETTP2982B25] [SMD]" (at 135.89 83.82 0) (effects (font (size 1.27 1.27)) (hide yes)))
 	)
 	(symbol
@@
 			)
 		)
+		(property "OEPS Description" "IC:   AUDIO SWITCH SPST DUAL   [FSA553UCX] [9-WLCSP]" (at 152.4 81.28 0) (effects (font (size 1.27 1.27)) (hide yes)))
 	)
 	(symbol
@@
 			)
 		)
+		(property "OEPS Description" "RESISTOR:   SMD 0402 301Ω ±0.1% 0.063W   [RT0402BRD07301RL] [SMD]" (at 129.54 90.17 0) (effects (font (size 1.27 1.27)) (hide yes)))
 	)
 )
