File: pcb/user-io.kicad_sch (KiCad schematic)
At the start: 26 parts, among them J4 FH12-24S-0.5SH(55), Q4 DMP3099L-7, Q6 DMG3418L, SW2 PEC12R-4222F-S0024, U150 SN74LVC1G14DBVR

Commit message: Change power switch
- Replace push button with rocker
- Added some notches to outside of PCB for aligning with enclosure
- Upgrade to KiCAD 9.0
Changed lines of the file:
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@@
 (kicad_sch
-	(version 20231120)
+	(version 20241209)
 	(generator "eeschema")
-	(generator_version "8.0")
+	(generator_version "9.0")
 	(paper "A4")
 	(title_block
@@
 		(members "~{RES}" "~{D/C}" "~{CS1}" "SCLK" "MOSI")
 	)
+	(text "Display:\nZJY130-2864KSWLG22"
+		(exclude_from_sim no)
+		(at 196.342 73.152 0)
+		(effects
+			(font
+				(size 1.27 1.27)
+			)
+			(justify left)
+			(href "https://cdn-shop.adafruit.com/product-files/5228/5223-ds.pdf")
+		)
+	)
+	(text "Knob:\nACCKMR1316NLT14"
+		(exclude_from_sim no)
+		(at 139.7 142.24 0)
+		(effects
+			(font
+				(size 1.27 1.27)
+			)
+			(href "https://www.vishay.com/docs/51101/acck.pdf")
+		)
+	)
 	(junction
 		(at 139.7 45.72)
@@
 		)
 	)
-	(text "Display:\nZJY130-2864KSWLG22"
-		(exclude_from_sim no)
-		(at 196.342 73.152 0)
-		(effects
-			(font
-				(size 1.27 1.27)
-			)
-			(justify left)
-			(href "https://cdn-shop.adafruit.com/product-files/5228/5223-ds.pdf")
-		)
-	)
-	(text "Knob:\nACCKMR1316NLT14"
-		(exclude_from_sim no)
-		(at 139.7 142.24 0)
-		(effects
-			(font
-				(size 1.27 1.27)
-			)
-			(href "https://www.vishay.com/docs/51101/acck.pdf")
-		)
-	)
 	(label "VBAT"
 		(at 187.96 45.72 180)
-		(fields_autoplaced yes)
 		(effects
 			(font
@@
 	(label "~{CS1}"
 		(at 173.99 53.34 0)
-		(fields_autoplaced yes)
 		(effects
 			(font
@@
 	(label "~{D{slash}C}"
 		(at 173.99 58.42 0)
-		(fields_autoplaced yes)
 		(effects
 			(font
@@
 	(label "SCLK"
 		(at 173.99 60.96 0)
-		(fields_autoplaced yes)
 		(effects
 			(font
@@
 	(label "MOSI"
 		(at 173.99 63.5 0)
-		(fields_autoplaced yes)
 		(effects
 			(font
@@
 	(label "VBAT"
 		(at 114.3 64.77 0)
-		(fields_autoplaced yes)
 		(effects
 			(font
@@
 	(label "~{RES}"
 		(at 173.99 55.88 0)
-		(fields_autoplaced yes)
 		(effects
 			(font
@@
 		(shape output)
 		(at 106.68 151.13 180)
-		(fields_autoplaced yes)
 		(effects
 			(font
@@
 		(shape input)
 		(at 170.18 50.8 180)
-		(fields_autoplaced yes)
 		(effects
 			(font
@@
 		(shape output)
 		(at 85.09 151.13 180)
-		(fields_autoplaced yes)
 		(effects
 			(font
@@
 		(shape input)
 		(at 69.85 63.5 180)
-		(fields_autoplaced yes)
 		(effects
 			(font
@@
 		(shape output)
 		(at 208.28 130.81 0)
-		(fields_autoplaced yes)
-		(effects
-			(font
+		(effects
+			(font

Commit message: Added module detect signal
- 100k pullup to VCC next to i2c bus that can be pulled down by module
  to assert its presence
Other:
- company: (none) -> Open Ephys, Inc
- title: (none) -> Extracellular Electrophysiology Test Board
Changed lines of the file:
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@@
 	(paper "A4")
 	(title_block
-		(rev "B")
+		(title "Extracellular Electrophysiology Test Board")
+		(rev "C")
+		(company "Open Ephys, Inc")
 		(comment 1 "Jonathan P. Newman")
 	)
