File: pcb/user-io.kicad_sch (KiCad schematic)
At the start: 26 parts, among them J4 FH12-24S-0.5SH(55), Q4 DMP3099L-7, Q6 DMG3418L, SW2 PEC12R-4222F-S0024, U150 SN74LVC1G14DBVR

Commit message: Fix J4 value
- FH12-16S-0.5SH(55) instead of FH12-24S-0.5SH(55)
Parts:
- J4: value FH12-24S-0.5SH(55) -> FH12-16S-0.5SH(55)
Changed lines of the file:
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@@
 			)
 		)
-		(property "Value" "FH12-24S-0.5SH(55)"
+		(property "Value" "FH12-16S-0.5SH(55)"
 			(at 195.58 56.2355 0)
 			(effects

Commit message: Mirror connections on J4
- The schematic presented on OLED datasheet was mirrored commpared to
  the connector's pin order. This fixes that.
Connections:
- net GND: now also J4.1 (Pin_1), J4.11 (Pin_11); no longer J4.16 (Pin_16), J4.6 (Pin_6)
- net MOSI: now also J4.5 (Pin_5); no longer J4.12 (Pin_12)
- net SCLK: now also J4.6 (Pin_6); no longer J4.11 (Pin_11)
- net VBAT: now also J4.12 (Pin_12); no longer J4.5 (Pin_5)
- net VCC: now also J4.10 (Pin_10); no longer J4.7 (Pin_7)
- net ~{CS1}: now also J4.9 (Pin_9); no longer J4.8 (Pin_8)
- net ~{D/C}: now also J4.7 (Pin_7); no longer J4.10 (Pin_10)
- net ~{RES}: now also J4.8 (Pin_8); no longer J4.9 (Pin_9)
- net at C305.1: now also J4.13 (Pin_13); no longer J4.4 (Pin_4)
- net at C305.2: now also J4.14 (Pin_14); no longer J4.3 (Pin_3)
- net at R277.1: now also J4.4 (Pin_4); no longer J4.13 (Pin_13)
- net at C306.1, C308.2: now also J4.2 (Pin_2); no longer J4.15 (Pin_15)
- net at C309.1: now also J4.3 (Pin_3); no longer J4.14 (Pin_14)
- net at C304.1: now also J4.15 (Pin_15); no longer J4.2 (Pin_2)
- net at C304.2: now also J4.16 (Pin_16); no longer J4.1 (Pin_1)
Other:
- note added: "NB: connector pinout is mirrored on datasheet"
- moved on the sheet: J4
Changed lines of the file:
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@@
 (kicad_sch
-	(version 20241209)
+	(version 20250114)
 	(generator "eeschema")
 	(generator_version "9.0")
@@
 	(text "Display:\nZJY130-2864KSWLG22"
 		(exclude_from_sim no)
-		(at 196.342 73.152 0)
+		(at 195.58 60.96 0)
 		(effects
 			(font
@@
 		)
 	)
+	(text "NB: connector pinout\nis mirrored on datasheet"
+		(exclude_from_sim no)
+		(at 195.58 66.04 0)
+		(effects
+			(font
+				(size 1.27 1.27)
+			)
+			(justify left)
+		)
+	)
 	(junction
 		(at 139.7 45.72)
@@
 		(color 0 0 0 0)
 	)
-	(junction
-		(at 193.04 80.01)
-		(diameter 0)
-		(color 0 0 0 0)
-	)
 	(bus_entry
 		(at 171.45 55.88)
@@
 	(wire
 		(pts
+			(xy 199.39 30.48) (xy 199.39 35.56)
+		)
+		(stroke
+			(width 0)
+			(type default)
+		)
+	)
+	(wire
+		(pts
 			(xy 100.33 64.77) (xy 109.22 64.77)
 		)
@@
 	(wire
 		(pts
+			(xy 193.04 30.48) (xy 199.39 30.48)
+		)
+		(stroke
+			(width 0)
+			(type default)
+		)
+	)
+	(wire
+		(pts
 			(xy 180.34 78.74) (xy 180.34 82.55)
 		)
@@
 	(wire
 		(pts
-			(xy 186.69 73.66) (xy 186.69 80.01)
+			(xy 186.69 73.66) (xy 186.69 82.55)
 		)
 		(stroke
@@
 		)
 	)
-	(wire
-		(pts
-			(xy 193.04 80.01) (xy 193.04 82.55)
-		)
-		(stroke
-			(width 0)
-			(type default)
-		)
-	)
 	(bus
 		(pts
@@
 	(wire
 		(pts
-			(xy 193.04 78.74) (xy 193.04 80.01)
-		)
-		(stroke
-			(width 0)
-			(type default)
-		)
-	)
-	(wire
-		(pts
 			(xy 87.63 148.59) (xy 87.63 151.13)
 		)
@@
 	(wire
 		(pts
-			(xy 186.69 80.01) (xy 193.04 80.01)
-		)
-		(stroke
-			(width 0)
-			(type default)
-		)
-	)
-	(wire
-		(pts
 			(xy 81.28 54.61) (xy 85.09 54.61)
 		)
@@
 	(symbol
 		(lib_id "power:GND")
-		(at 193.04 82.55 0)
+		(at 186.69 82.55 0)
 		(mirror y)
 		(unit 1)
@@
 		(fields_autoplaced yes)
 		(property "Reference" "#PWR0791"
-			(at 193.04 88.9 0)
+			(at 186.69 88.9 0)
 			(effects
 				(font
@@
 		)
 		(property "Value" "GND"
-			(at 193.04 87.63 0)
+			(at 186.69 87.63 0)
 			(effects
 				(font
@@
 		)
 		(property "Footprint" ""
-			(at 193.04 82.55 0)
+			(at 186.69 82.55 0)
 			(effects
 				(font
@@
 		)
 		(property "Datasheet" ""
-			(at 193.04 82.55 0)
+			(at 186.69 82.55 0)
 			(effects
 				(font
@@
 		)
 		(property "Description" "Power symbol creates a global label with name \"GND\" , ground"
-			(at 193.04 82.55 0)
+			(at 186.69 82.55 0)
 			(effects
 				(font
@@
 	)
 	(symbol
+		(lib_id "power:GND")
+		(at 199.39 35.56 0)
+		(mirror y)
+		(unit 1)
+		(exclude_from_sim no)
+		(in_bom yes)
+		(on_board yes)
+		(dnp no)
+		(fields_autoplaced yes)
+		(property "Reference" "#PWR0793"
+			(at 199.39 41.91 0)
+			(effects
+				(font
+					(size 1.27 1.27)
+				)
+				(hide yes)
+			)
+		)
+		(property "Value" "GND"
+			(at 199.39 40.64 0)
+			(effects
+				(font
+					(size 1.27 1.27)
+				)
+			)
+		)
+		(property "Footprint" ""
+			(at 199.39 35.56 0)
+			(effects
+				(font
+					(size 1.27 1.27)
+				)
+				(hide yes)
+			)
+		)
+		(property "Datasheet" ""
+			(at 199.39 35.56 0)
+			(effects
+				(font
+					(size 1.27 1.27)
+				)
+				(hide yes)
+			)
+		)
+		(property "Description" "Power symbol creates a global label with name \"GND\" , ground"
+			(at 199.39 35.56 0)
+			(effects
+				(font
+					(size 1.27 1.27)
+				)
+				(hide yes)
+			)
+		)
+		(pin "1"
+		)
+		(instances
+			(project "ephys-test-board"
+				(path "/ffaa6ffd-73fa-4da3-9ff1-78fa7369281f/0564b576-016f-4657-a76f-817e9e3dffb1"
+					(reference "#PWR0793")
+					(unit 1)
+				)
+			)
+		)
+	)
+	(symbol
 		(lib_id "Device:C")
 		(at 180.34 74.93 0)
@@
 	(symbol
 		(lib_id "Connector_Generic_MountingPin:Conn_01x16_MountingPin")
-		(at 193.04 53.34 0)
+		(at 193.04 55.88 0)
+		(mirror x)
 		(unit 1)
 		(exclude_from_sim no)
@@
 		(on_board yes)
 		(dnp no)
-		(fields_autoplaced yes)
 		(property "Reference" "J4"
-			(at 195.58 53.6955 0)
+			(at 195.58 55.5245 0)
 			(effects
 				(font
@@
 		)
 		(property "Value" "FH12-16S-0.5SH(55)"
-			(at 195.58 56.2355 0)
+			(at 195.58 52.9845 0)
 			(effects
 				(font
@@
 		)
 		(property "Footprint" "Connector_FFC-FPC:Hirose_FH12-16S-0.5SH_1x16-1MP_P0.50mm_Horizontal"
-			(at 193.04 53.34 0)
+			(at 193.04 55.88 0)
 			(effects
 				(font
@@
 		)
 		(property "Datasheet" "~"
-			(at 193.04 53.34 0)
+			(at 193.04 55.88 0)
 			(effects
 				(font
@@
 		)
 		(property "Description" "Generic connectable mounting pin connector, single row, 01x16, script generated (kicad-library-utils/schlib/autogen/connector/)"
-			(at 193.04 53.34 0)
+			(at 193.04 55.88 0)
 			(effects
 				(font
@@
 		)
 		(property "Datasheet1" ""
-			(at 193.04 53.34 0)
+			(at 193.04 55.88 0)
 			(effects
 				(font
@@
 		)
 		(property "Part No." ""
-			(at 193.04 53.34 0)
+			(at 193.04 55.88 0)
 			(effects
 				(font

Commit message: Added OEPS PN.
Co-Authored-By: David Palma <78764277+davidpalma666@users.noreply.github.com>
Parts:
- C293, C294: MPN (none) -> C1005X7R1E104K050BB; OEPSPN (none) -> OEPS010050
- C296, C303: MPN (none) -> GRM155R71E103KA01D; OEPSPN (none) -> OEPS010067
- C300, C302, C304, C305, C308: MPN (none) -> CL10A105KA8NNNC; OEPSPN (none) -> OEPS010022
- C301, C306, C309: MPN (none) -> CL31B475KOHNNNE; OEPSPN (none) -> OEPS010081
- J4: MPN (none) -> FH12-16S-0.5SH(55); OEPSPN (none) -> OEPS070104
- Q4: MPN (none) -> DMP3099L-7; OEPSPN (none) -> OEPS060020
- Q6: MPN (none) -> DMG3418L-7; OEPSPN (none) -> OEPS060019
- R269, R279, R280, R281, R282: MPN (none) -> CRCW040210K0FKED; OEPSPN (none) -> OEPS020030
- R277: MPN (none) -> RC0402FR-13680KL; OEPSPN (none) -> OEPS020176
- R278: MPN (none) -> CRCW04021K00FKED; OEPSPN (none) -> OEPS020027
- R286, R287: MPN (none) -> ERJ-2RKF4702X; OEPSPN (none) -> OEPS020017
- SW2: MPN (none) -> PEC12R-4222F-S0024; OEPSPN (none) -> OEPS070113
- U150: MPN (none) -> SN74LVC1G14DBVR; OEPSPN (none) -> OEPS080160

Commit message: Use 1.25V reference voltage for electrode test signal
- This prevents large AC component when channel switch occurs.
- Previously the attenuator reference and nomimal electrode signals were
  both ground. Since the test signal is centered arround 1.25V, there
  the test signal is effectively a 1.25V square wave + the indented
  signal. The square waves edges were readily passed through the AC
  coupling capacitor.
- Add LCSC numbers to all required components for assembly.
Parts:
- C293, C294: LCSC (none) -> C105883; Voltage (none) -> 25V
- C296, C303: LCSC (none) -> C60133; Voltage (none) -> 50V
- C300, C302, C304, C305, C308: LCSC (none) -> C5673
- C301, C306, C309: LCSC (none) -> C51205
- J4: LCSC (none) -> C262665
- Q4: LCSC (none) -> C155244
- Q6: value DMG3418L -> DMG3418L-7; LCSC (none) -> C151026
- R269, R279, R280, R281, R282: LCSC (none) -> C60490
- R277: LCSC (none) -> C2909377
- R278: LCSC (none) -> C106235
- R286, R287: LCSC (none) -> C93943
- SW2: value PEC12R-4222F-S0024 -> PEC12R-4220F-S0024; LCSC (none) -> C18164805
- U150: LCSC (none) -> C7835
