File: pcb/user-io.kicad_sch (KiCad schematic)
At the start: 26 parts, among them J4 FH12-16S-0.5SH(55), Q4 DMP3099L-7, Q6 DMG3418L-7, SW2 PEC12R-4220F-S0024, U150 SN74LVC1G14DBVR

Commit message: Implmenent bipolar test signal
- Generate internal negative rail
- Shift DAC output by VREF/2
- Replace analog switches with depletion mode switches to allow negative
  signals
- DC couple electrode inputs
Parts:
- renumbered C296 to C116, C300 to C117, C303 to C118, C301 to C119, C302 to C120, C309 to C121, C305 to C122, C306 to C123, C304 to C124, C294 to C125, C308 to C126, C293 to C127, J4 to J8, Q6 to Q4, Q4 to Q5, R287 to R282, R286 to R283, R279 to R284, R281 to R285, R280 to R286, R282 to R287, R277 to R288, R269 to R289, R278 to R290, SW2 to SW4, U150 to U93

Commit message: Revision G candidate
- Fix flipped power/ground connections on U84
- VCC is now 3.0V
- Address issues with parasitic voltage feedthrough on FSA533
- Completely redesign test signal analog section with much
  improved noise, THD, etc and implicit low THD input protection on the
  external input.
Parts:
- R290: LCSC C106235 -> (none); Tolerance (none) -> 0.1%
Changed lines of the file:
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@@
 	(title_block
 		(title "Extracellular Electrophysiology Test Board")
-		(rev "F")
+		(rev "G")
 		(company "Open Ephys, Inc")
 		(comment 1 "Jonathan P. Newman")
@@
 			)
 		)
-		(property "Tolerance" ""
+		(property "Tolerance" "0.1%"
 			(at 163.83 130.81 0)
 			(effects
@@
 					(size 1.27 1.27)
 				)
+				(hide yes)
 			)
 		)
@@
 			)
 		)
-		(property "LCSC" "C106235"
+		(property "LCSC" ""
 			(at 163.83 130.81 90)
 			(effects

Commit message: Update PCB component part numbers
Replace and fill missing MPN and OEPSPN properties.
Parts:
- R290: MPN CRCW04021K00FKED -> ERA-1AEB102C; OEPSPN OEPS020027 -> OEPS020189
- SW4: MPN PEC12R-4222F-S0024 -> PEC12R-4220F-S0024; OEPSPN OEPS070113 -> OEPS100076
Changed lines of the file:
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@@
 			)
 		)
-		(property "MPN" "CRCW04021K00FKED"
+		(property "MPN" "ERA-1AEB102C"
 			(at 163.83 130.81 0)
 			(effects
@@
 			)
 		)
-		(property "OEPSPN" "OEPS020027"
+		(property "OEPSPN" "OEPS020189"
 			(at 163.83 130.81 0)
 			(effects
@@
 			)
 		)
-		(property "MPN" "PEC12R-4222F-S0024"
+		(property "MPN" "PEC12R-4220F-S0024"
 			(at 139.7 133.35 0)
 			(effects
@@
 			)
 		)
-		(property "OEPSPN" "OEPS070113"
+		(property "OEPSPN" "OEPS100076"
 			(at 139.7 133.35 0)
 			(effects

Commit message: Rev. G production candidate
- Finished LCSC part numbers
- Generated final gerbers
Parts:
- R290: LCSC (none) -> C852624
Changed lines of the file:
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@@
 			)
 		)
-		(property "LCSC" ""
+		(property "LCSC" "C852624"
 			(at 163.83 130.81 90)
 			(effects

Commit message: Minor BOM fix before production
Update the 1k 0402 resistor footprint/PN across BOM and schematics.
Parts:
- R290: LCSC C852624 -> C2073397; MPN ERA-1AEB102C -> RG1005P-102-B-T5; OEPSPN OEPS020189 -> OEPS020219
Changed lines of the file:
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@@
 			)
 		)
-		(property "MPN" "ERA-1AEB102C"
+		(property "MPN" "RG1005P-102-B-T5"
 			(at 163.83 130.81 0)
 			(effects
@@
 			)
 		)
-		(property "OEPSPN" "OEPS020189"
+		(property "OEPSPN" "OEPS020219"
 			(at 163.83 130.81 0)
 			(effects
@@
 			)
 		)
-		(property "LCSC" "C852624"
+		(property "LCSC" "C2073397"
 			(at 163.83 130.81 90)
 			(effects
