File: pcb/headstage-io.kicad_sch (KiCad schematic)
At the start: 4 parts, among them J2 BTE-040-02-F-D-A, J3 BTE-040-02-F-D-A

Commit message: Routing nearly complete
- Power switch is too tall I think
Parts:
- J2, J3: value BTE-040-02-F-D-A -> BTE-040-03-L-D-A
Changed lines of the file:
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@@
 			)
 		)
-		(property "Value" "BTE-040-02-F-D-A"
+		(property "Value" "BTE-040-03-L-D-A"
 			(at 87.63 40.64 0)
 			(effects
@@
 		)
 		(property "Description" "Generic connector, double row, 02x40, odd/even pin numbering scheme (row 1 odd numbers, row 2 even numbers), script generated (kicad-library-utils/schlib/autogen/connector/)"
+			(at 88.9 92.71 0)
+			(effects
+				(font
+					(size 1.27 1.27)
+				)
+				(hide yes)
+			)
+		)
+		(property "Voltage" ""
 			(at 88.9 92.71 0)
 			(effects
@@
 			)
 		)
-		(property "Value" "BTE-040-02-F-D-A"
+		(property "Value" "BTE-040-03-L-D-A"
 			(at 193.04 40.64 0)
 			(effects
@@
 		)
 		(property "Description" "Generic connector, double row, 02x40, odd/even pin numbering scheme (row 1 odd numbers, row 2 even numbers), script generated (kicad-library-utils/schlib/autogen/connector/)"
+			(at 194.31 92.71 0)
+			(effects
+				(font
+					(size 1.27 1.27)
+				)
+				(hide yes)
+			)
+		)
+		(property "Voltage" ""
 			(at 194.31 92.71 0)
 			(effects
@@
 			)
 		)
+		(property "Voltage" ""
+			(at 114.3 134.62 0)
+			(effects
+				(font
+					(size 1.27 1.27)
+				)
+				(hide yes)
+			)
+		)
 		(pin "1"
 		)
@@
 			(at 123.19 134.62 0)
 			(effects
+				(font
+					(size 1.27 1.27)
+				)
+				(hide yes)
+			)
+		)
+		(property "Voltage" ""
+			(at 123.19 134.62 0)
+			(effects

Commit message: Added module detect signal
- 100k pullup to VCC next to i2c bus that can be pulled down by module
  to assert its presence
Parts:
- added R288: 100k, Resistor_SMD:R_0402_1005Metric, symbol Device:R_US
- R284, R285: now not fitted
Connections:
- net GND: no longer J2.78 (Pin_78)
- net VCC: now also R288.1
- new net Detect: J2.78 (Pin_78), R288.2
