File: pcb/ephys-test-board.kicad_pcb (KiCad board)
At the start: 4 copper layers, 150 x 120 mm, 567 parts, among them J1 10129383-910002ALF, J2 BM03B-SRSS-TB, J3 BTE-040-03-L-D-A, J4 BTE-040-03-L-D-A, J5 731000105, J6 USB4105-GF-A, J7 S2B-PH-SM4-TB, J8 FH12-16S-0.5SH(55), Q1 DMP3099L-7, Q2 DMG3418L-7, Q3 DMG3418L-7, Q4 DMG3418L-7, Q5 DMP3099L-7, SW1 PTS645VH83-2 LFS, SW2 TS04-66-50-BK-160-SMT, SW3 400MSP1R6BLKM6QE, SW4 PEC12R-4220F-S0024, U1 W25Q128JVSIQ, U10 FSA553UCX, U11 FSA553UCX, U12 SN74HC595PWR, U13 FSA553UCX, U14 FSA553UCX, U15 FSA553UCX, U16 FSA553UCX, U17 SN74HC595PWR, U18 FSA553UCX, U19 FSA553UCX, U2 SC0914(13), U20 FSA553UCX, U21 FSA553UCX, U22 SN74HC595PWR, U23 FSA553UCX, U24 FSA553UCX, U25 FSA553UCX, U26 FSA553UCX, U27 SN74HC595PWR, U28 FSA553UCX, U29 FSA553UCX, U3 FSA553UCX, U30 FSA553UCX, U31 FSA553UCX, U32 SN74HC595PWR, U33 FSA553UCX, U34 FSA553UCX, U35 FSA553UCX, U36 FSA553UCX, U37 SN74HC595PWR, U38 FSA553UCX, U39 FSA553UCX, U4 FSA553UCX, U40 FSA553UCX, U41 FSA553UCX, U42 SN74HC595PWR, U43 FSA553UCX, U44 FSA553UCX, U45 FSA553UCX, U46 FSA553UCX, U47 SN74HC595PWR, U48 FSA553UCX, U49 FSA553UCX, U5 FSA553UCX, U50 FSA553UCX, U51 FSA553UCX, U52 SN74HC595PWR, U53 FSA553UCX, U54 FSA553UCX, U55 FSA553UCX, U56 FSA553UCX, U57 SN74HC595PWR, U58 FSA553UCX, U59 FSA553UCX, U6 FSA553UCX, U60 FSA553UCX, U61 FSA553UCX, U62 SN74HC595PWR, U63 FSA553UCX, U64 FSA553UCX, U65 FSA553UCX, U66 FSA553UCX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

Commit message: Update to KiCAD v10 and fix BOM
Updated BOM according to the design being produced.
Parts:
- R100, R101, R102, R107, R108, R109, R11, R110, R115, R116, R117, R118, R12, R123, R124, R125, R126, R13, R131, R132, R133, R134, R139, R14, R140, R141, R142, R147, R148, R149, R150, R155, R156, R157, R158, R163, R164, R165, R166, R171, R172, R173, R174, R179, R180, R181, R182, R187, R188, R189, R19, R190, R195, R196, R197, R198, R20, R203, R204, R205, R206, R21, R211, R212, R213, R214, R219, R22, R220, R221, R222, R227, R228, R229, R230, R235, R236, R237, R238, R243, R244, R245, R246, R251, R252, R253, R254, R259, R260, R261, R262, R27, R28, R29, R30, R35, R36, R37, R38, R43, R44, R45, R46, R51, R52, R53, R54, R59, R60, R61, R62, R67, R68, R69, R70, R75, R76, R77, R78, R83, R84, R85, R86, R91, R92, R93, R94, R99: value 200R -> 301R
- R103, R104, R105, R106, R111, R112, R113, R114, R119, R120, R121, R122, R127, R128, R129, R130, R135, R136, R137, R138, R143, R144, R145, R146, R15, R151, R152, R153, R154, R159, R16, R160, R161, R162, R167, R168, R169, R17, R170, R175, R176, R177, R178, R18, R183, R184, R185, R186, R191, R192, R193, R194, R199, R200, R201, R202, R207, R208, R209, R210, R215, R216, R217, R218, R223, R224, R225, R226, R23, R231, R232, R233, R234, R239, R24, R240, R241, R242, R247, R248, R249, R25, R250, R255, R256, R257, R258, R26, R263, R264, R265, R266, R31, R32, R33, R34, R39, R40, R41, R42, R47, R48, R49, R50, R55, R56, R57, R58, R63, R64, R65, R66, R71, R72, R73, R74, R79, R80, R81, R82, R87, R88, R89, R90, R95, R96, R97, R98: value 19.8k -> 29.8k
