File: pcb/ephys-test-board.kicad_pcb (KiCad board)
At the start: 4 copper layers, 150 x 120 mm, 567 parts, among them J1 10129383-910002ALF, J2 BM03B-SRSS-TB, J3 BTE-040-03-L-D-A, J4 BTE-040-03-L-D-A, J5 731000105, J6 USB4105-GF-A, J7 S2B-PH-SM4-TB, J8 FH12-16S-0.5SH(55), Q1 DMP3099L-7, Q2 DMG3418L-7, Q3 DMG3418L-7, Q4 DMG3418L-7, Q5 DMP3099L-7, SW1 PTS645VH83-2 LFS, SW2 TS04-66-50-BK-160-SMT, SW3 400MSP1R6BLKM6QE, SW4 PEC12R-4220F-S0024, U1 W25Q128JVSIQ, U10 FSA553UCX, U11 FSA553UCX, U12 SN74HC595PWR, U13 FSA553UCX, U14 FSA553UCX, U15 FSA553UCX, U16 FSA553UCX, U17 SN74HC595PWR, U18 FSA553UCX, U19 FSA553UCX, U2 SC0914(13), U20 FSA553UCX, U21 FSA553UCX, U22 SN74HC595PWR, U23 FSA553UCX, U24 FSA553UCX, U25 FSA553UCX, U26 FSA553UCX, U27 SN74HC595PWR, U28 FSA553UCX, U29 FSA553UCX, U3 FSA553UCX, U30 FSA553UCX, U31 FSA553UCX, U32 SN74HC595PWR, U33 FSA553UCX, U34 FSA553UCX, U35 FSA553UCX, U36 FSA553UCX, U37 SN74HC595PWR, U38 FSA553UCX, U39 FSA553UCX, U4 FSA553UCX, U40 FSA553UCX, U41 FSA553UCX, U42 SN74HC595PWR, U43 FSA553UCX, U44 FSA553UCX, U45 FSA553UCX, U46 FSA553UCX, U47 SN74HC595PWR, U48 FSA553UCX, U49 FSA553UCX, U5 FSA553UCX, U50 FSA553UCX, U51 FSA553UCX, U52 SN74HC595PWR, U53 FSA553UCX, U54 FSA553UCX, U55 FSA553UCX, U56 FSA553UCX, U57 SN74HC595PWR, U58 FSA553UCX, U59 FSA553UCX, U6 FSA553UCX, U60 FSA553UCX, U61 FSA553UCX, U62 SN74HC595PWR, U63 FSA553UCX, U64 FSA553UCX, U65 FSA553UCX, U66 FSA553UCX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

Commit message: Added 'Description' to all the components
Updated PCB accordingly.
Configured files for manufacturing generation according to standards.
Parts:
- J5: value 731000105 -> 0731000105
